File: Circuit/Roll Swarm/Roll Swarm.brd (EAGLE design)
At the start: 23.5 x 38.1 mm, 18 parts, among them IC1 MCP1703CB, J7 CORTEX_DEBUG_SMD, U1 MDBT50Q-1MV2, U5 74AHCT2G125

Commit message: Adding new board-mount on/off switch.
Parts:
- removed J5: (no value), SparkFun-Connectors:1X02_XTRA_BIG
- added S1: EG2208, EG2208:SW_EG2208
- moved IC1 10.9 mm to (24.8, 30.5)
- moved R2 10.4 mm to (24.8, 26.7)
- moved U5 10.2 mm to (25.1, 22.5)
- moved D3 9.53 mm to (24.8, 24.4)
Connections:
- net VBAT: now also S1.6; no longer J5.1
- net VBAT_RAW: now also S1.3; no longer J5.2
